File: Receiving loop/RX Loop/RX Loop.sch (KiCad schematic (older format))
At the start: 40 parts, among them IC1 GALI-74, IC2 GALI-74, J1 VCC, K1 G5V-1, K2 G5V-1, T1 4T Primary 3T Secondary #24, U1 L7812

Commit message: Fixed footprint label for U1
Parts:
- U1: value L7812 -> L7805
Changed lines of the file:
@@
 P 4660 5230
 F 0 "U1" H 4660 5472 50  0000 C CNN
-F 1 "L7812" H 4660 5381 50  0000 C CNN
+F 1 "L7805" H 4660 5381 50  0000 C CNN
 F 2 "Package_TO_SOT_THT:TO-220F-3_Vertical" H 4685 5080 50  0001 L CIN
 F 3 "http://www.st.com/content/ccc/resource/technical/document/datasheet/41/4f/b3/b0/12/d4/47/88/CD00000444.pdf/files/CD00000444.pdf/jcr:content/translations/en.CD00000444.pdf" H 4660 5180 50  0001 C CNN

Commit message: Updating changes. Cleaning up repo.wq
Parts:
- K1, K2: value G5V-1 -> G5V-1 DC9
- R1, R5: value 560 Ohms -> 560 Ohms 1%
- R6, R7: value 4.3 Ohms -> 4.3 Ohms 1%
- T1: value 4T Primary 3T Secondary #24 -> 5T Primary 4T Secondary #24
- U1: value L7805 -> L7809
Connections:
- net labels added: +9V
- net labels removed: +12V
Changed lines of the file:
@@
 P 2460 2430
 F 0 "R5" H 2519 2476 50  0000 L CNN
-F 1 "560 Ohms" H 2519 2385 50  0000 L CNN
+F 1 "560 Ohms 1%" H 2519 2385 50  0000 L CNN
 F 2 "w8tam_footprints:RNF14FTD1K00" H 2460 2430 50  0001 C CNN
 F 3 "~" H 2460 2430 50  0001 C CNN
@@
 P 2460 3080
 F 0 "R1" H 2519 3126 50  0000 L CNN
-F 1 "560 Ohms" H 2519 3035 50  0000 L CNN
+F 1 "560 Ohms 1%" H 2519 3035 50  0000 L CNN
 F 2 "w8tam_footprints:RNF14FTD1K00" H 2460 3080 50  0001 C CNN
 F 3 "~" H 2460 3080 50  0001 C CNN
@@
 P 3160 2180
 F 0 "R7" V 2964 2180 50  0000 C CNN
-F 1 "4.3 Ohms" V 3055 2180 50  0000 C CNN
+F 1 "4.3 Ohms 1%" V 3055 2180 50  0000 C CNN
 F 2 "w8tam_footprints:RNF14FTD1K00" H 3160 2180 50  0001 C CNN
 F 3 "~" H 3160 2180 50  0001 C CNN
@@
 P 3110 3430
 F 0 "R6" H 3169 3476 50  0000 L CNN
-F 1 "4.3 Ohms" H 3169 3385 50  0000 L CNN
+F 1 "4.3 Ohms 1%" H 3169 3385 50  0000 L CNN
 F 2 "w8tam_footprints:RNF14FTD1K00" H 3110 3430 50  0001 C CNN
 F 3 "~" H 3110 3430 50  0001 C CNN
@@
 P 8560 2580
 F 0 "T1" H 8560 2961 50  0000 C CNN
-F 1 "4T Primary 3T Secondary #24" H 8560 2870 50  0000 C CNN
+F 1 "5T Primary 4T Secondary #24" H 8560 2870 50  0000 C CNN
 F 2 "w8tam_footprints:Binocular" H 8560 2580 50  0001 C CNN
 F 3 "~" H 8560 2580 50  0001 C CNN
@@
 P 4660 5230
 F 0 "U1" H 4660 5472 50  0000 C CNN
-F 1 "L7805" H 4660 5381 50  0000 C CNN
+F 1 "L7809" H 4660 5381 50  0000 C CNN
 F 2 "Package_TO_SOT_THT:TO-220F-3_Vertical" H 4685 5080 50  0001 L CIN
 F 3 "http://www.st.com/content/ccc/resource/technical/document/datasheet/41/4f/b3/b0/12/d4/47/88/CD00000444.pdf/files/CD00000444.pdf/jcr:content/translations/en.CD00000444.pdf" H 4660 5180 50  0001 C CNN
@@
 P 1815 3130
 F 0 "K2" V 2325 3130 50  0000 C CNN
-F 1 "G5V-1" V 2265 3130 50  0000 C CNN
+F 1 "G5V-1 DC9" V 2265 3130 50  0000 C CNN
 F 2 "Relay_THT:Relay_SPDT_Omron_G5V-1" H 2945 3100 50  0001 C CNN
 F 3 "http://omronfs.omron.com/en_US/ecb/products/pdf/en-g5v_1.pdf" H 1815 3130 50  0001 C CNN
@@
 	0    1    1    0
 $EndComp
-$Comp
-L power:+12V #PWR0122
-U 1 1 60647163
-P 6845 5230
-F 0 "#PWR0122" H 6845 5080 50  0001 C CNN
-F 1 "+12V" H 6860 5403 50  0000 C CNN
-F 2 "" H 6845 5230 50  0001 C CNN
-F 3 "" H 6845 5230 50  0001 C CNN
-	1    6845 5230
-	1    0    0    -1
-$EndComp
-Connection ~ 6845 5230
-Wire Wire Line
-	6845 5230 7260 5230
-$Comp
-L power:+12V #PWR0123
-U 1 1 60649F82
-P 2115 2930
-F 0 "#PWR0123" H 2115 2780 50  0001 C CNN
-F 1 "+12V" V 2130 3058 50  0000 L CNN
-F 2 "" H 2115 2930 50  0001 C CNN
-F 3 "" H 2115 2930 50  0001 C CNN
-	1    2115 2930
-	0    1    1    0
-$EndComp
-Wire Wire Line
-	6410 5230 6845 5230
 Wire Wire Line
 	2460 3430 3010 3430
@@
 $EndComp
 $Comp
-L power:+12V #PWR0124
-U 1 1 6067BADF
-P 1500 1685
-F 0 "#PWR0124" H 1500 1535 50  0001 C CNN
-F 1 "+12V" V 1515 1813 50  0000 L CNN
-F 2 "" H 1500 1685 50  0001 C CNN
-F 3 "" H 1500 1685 50  0001 C CNN
-	1    1500 1685
-	0    -1   -1   0
-$EndComp
-$Comp
 L Device:D D5
 U 1 1 6040A791
@@
 P 1800 1885
 F 0 "K1" V 2367 1885 50  0000 C CNN
-F 1 "G5V-1" V 2276 1885 50  0000 C CNN
+F 1 "G5V-1 DC9" V 2276 1885 50  0000 C CNN
 F 2 "Relay_THT:Relay_SPDT_Omron_G5V-1" H 2930 1855 50  0001 C CNN
 F 3 "http://omronfs.omron.com/en_US/ecb/products/pdf/en-g5v_1.pdf" H 1800 1885 50  0001 C CNN
@@
 Wire Wire Line
 	2115 2930 1980 2660
-Connection ~ 2115 2930
 $Comp
 L power:GND #PWR0120
@@
 Wire Wire Line
 	1500 1685 1605 1410
-Connection ~ 1500 1685
 Text Notes 7410 7485 0    50   ~ 0
 MFJ-1886 Loop modified by W8TAM
@@
 Wire Wire Line
 	7860 2780 7760 2780
+$Comp
+L power:+9V #PWR?
+U 1 1 60CFE8B8
+P 2115 2930
+F 0 "#PWR?" H 2115 2780 50  0001 C CNN
+F 1 "+9V" V 2130 3058 50  0000 L CNN
+F 2 "" H 2115 2930 50  0001 C CNN
+F 3 "" H 2115 2930 50  0001 C CNN
+	1    2115 2930
+	0    1    1    0
+$EndComp
+Connection ~ 2115 2930
+$Comp
+L power:+9V #PWR?
+U 1 1 60D0342A
+P 1500 1685
+F 0 "#PWR?" H 1500 1535 50  0001 C CNN
+F 1 "+9V" V 1515 1813 50  0000 L CNN
+F 2 "" H 1500 1685 50  0001 C CNN
+F 3 "" H 1500 1685 50  0001 C CNN
+	1    1500 1685
+	0    -1   -1   0
+$EndComp
+Connection ~ 1500 1685
+$Comp
+L power:+9V #PWR?
+U 1 1 60D076EB
+P 6665 5230
+F 0 "#PWR?" H 6665 5080 50  0001 C CNN
+F 1 "+9V" H 6680 5403 50  0000 C CNN
+F 2 "" H 6665 5230 50  0001 C CNN
+F 3 "" H 6665 5230 50  0001 C CNN
+	1    6665 5230
+	1    0    0    -1
+$EndComp
+Wire Wire Line
+	6410 5230 6665 5230
+Connection ~ 6665 5230
+Wire Wire Line
+	6665 5230 7260 5230
 $EndSCHEMATC

Commit message: Merged changes. Updated metadata.
Other:
- note added: "20210620"
Changed lines of the file:
@@
 Wire Wire Line
 	6665 5230 7260 5230
+Text Notes 8120 7635 0    50   ~ 0
+20210620
 $EndSCHEMATC
